Commit message: remove bicycle model something broken

File: steer_bot_description/urdf/steer_bot.urdf.xacro (robot description, xacro)
@@ -16,6 +16,6 @@
 <robot name="steer_bot" xmlns:xacro="http://wiki.ros.org/xacro">
   <!-- Include xacro for inertials, materials and wheels -->
-  <xacro:include filename="$(find steer_bot_description)/urdf/wheel.xacro"/>
-  <xacro:property name="robot_namespace" value="/steer_bot"/>
+  <xacro:include filename="$(find steer_bot_description)/urdf/wheel.xacro" />
+  <xacro:property name="robot_namespace" value="/steer_bot" />
   <!-- Gazebo plugins -->
   <gazebo>
@@ -29,13 +29,13 @@
   </gazebo>
   <!-- Math constants -->
-  <xacro:property name="deg_to_rad" value="0.01745329251994329577"/>
+  <xacro:property name="deg_to_rad" value="0.01745329251994329577" />
   <!-- Robot base dimensions -->
-  <xacro:property name="base_length" value="0.5" />
-  <xacro:property name="base_width" value="0.3" />
-  <xacro:property name="base_height" value="0.1" />
+  <xacro:property name="base_length" value="3.6" />
+  <xacro:property name="base_width" value="2.5" />
+  <xacro:property name="base_height" value="0.25" />
   <xacro:property name="base_mass" value="5" />
   <!-- Wheel link dimensions -->
-  <xacro:property name="wheel_radius" value="0.1" />
-  <xacro:property name="wheel_thickness" value="0.08" />
+  <xacro:property name="wheel_radius" value="0.5" />
+  <xacro:property name="wheel_thickness" value="0.3" />
   <xacro:property name="wheel_mass" value="1" />
   <!-- Steering link dimensions -->
@@ -47,90 +47,42 @@
   <xacro:property name="steer_offset" value="0.02" />
   <!-- Base link -->
-  <link name="base_link">
+  <link name="base_link"></link>
+  <!-- A fixed joint for to connect base and chassis links -->
+  <joint name="base_link" type="fixed">
+    <origin xyz="0 0 0" rpy="0 0 0" />
+    <parent link="base_link" />
+    <child link="chassis_link" />
+  </joint>
+  <!-- Dummy Chassis link -->
+  <link name="chassis_link">
     <visual>
-      <origin xyz="0 0 0" rpy="0 0 0"/>
+      <origin xyz="0 0 0" rpy="0 0 0" />
       <geometry>
-        <box size="${base_length} ${base_width} ${base_height}"/>
+        <box size="${base_length} ${base_width} ${base_height}" />
       </geometry>
       <material name="green" />
     </visual>
     <collision>
-      <origin xyz="0 0 0" rpy="0 0 0"/>
+      <origin xyz="0 0 0" rpy="0 0 0" />
       <geometry>
-        <box size="${base_length} ${base_width} ${base_height}"/>
+        <box size="${base_length} ${base_width} ${base_height}" />
       </geometry>
     </collision>
-    <xacro:solid_cuboid_inertial
-        rpy="0 0 0" xyz="0 0 0"
-        mass="${base_mass}"
-        x="${base_length}" y="${base_width}" z="${base_height}" />
+    <xacro:solid_cuboid_inertial rpy="0 0 0" xyz="0 0 0" mass="${base_mass}" x="${base_length}" y="${base_width}" z="${base_height}" />
   </link>
   <!-- Front steer and rear wheel joints required for ackermann_steering_controller -->
-  <xacro:front_steer
-    name="front"
-    parent="base"
-    steer_radius="${steer_radius}"
-    steer_thickness="${steer_thickness}"
-    steer_mass="${steer_mass}"
-    base_length="${base_length}"
-    base_width="${base_width}"
-    axle_offset="${axle_offset}"
-    steer_height="${wheel_radius+steer_offset}">
-  </xacro:front_steer>
-  <xacro:rear_wheel
-    name="rear"
-    parent="base"
-    wheel_radius="${wheel_radius/4}"
-    wheel_thickness="${wheel_thickness/2}"
-    wheel_mass="${wheel_mass/32}">
-    <origin xyz="${-base_length/2+axle_offset} 0 0" rpy="${-90 * deg_to_rad} 0 0"/>
+  <xacro:front_steer name="front" parent="chassis" steer_radius="${steer_radius}" steer_thickness="${steer_thickness}" steer_mass="${steer_mass}" base_length="${base_length}" base_width="${base_width}" axle_offset="${axle_offset}" steer_height="${wheel_radius+steer_offset}"></xacro:front_steer>
+  <xacro:rear_wheel name="rear" parent="chassis" wheel_radius="${wheel_radius/4}" wheel_thickness="${wheel_thickness/2}" wheel_mass="${wheel_mass/32}">
+    <origin xyz="${-base_length/2+axle_offset} 0 0" rpy="${-90 * deg_to_rad} 0 0" />
   </xacro:rear_wheel>
   <!-- Steerable front wheels -->
-  <xacro:front_wheel_lr
-    name="front_right"
-    parent="base"
-    reflect="-1"
-    wheel_radius="${wheel_radius}"
-    wheel_thickness="${wheel_thickness}"
-    wheel_mass="${wheel_mass}"
-    steer_radius="${steer_radius}"
-    steer_thickness="${steer_thickness}"
-    steer_mass="${steer_mass}"
-    base_length="${base_length}"
-    base_width="${base_width}"
-    axle_offset="${axle_offset}"
-    steer_height="${wheel_radius+steer_offset}">
-  </xacro:front_wheel_lr>
-  <xacro:front_wheel_lr
-    name="front_left"
-    parent="base"
-    reflect="1"
-    wheel_radius="${wheel_radius}"
-    wheel_thickness="${wheel_thickness}"
-    wheel_mass="${wheel_mass}"
-    steer_radius="${steer_radius}"
-    steer_thickness="${steer_thickness}"
-    steer_mass="${steer_mass}"
-    base_length="${base_length}"
-    base_width="${base_width}"
-    axle_offset="${axle_offset}"
-    steer_height="${wheel_radius+steer_offset}">
-  </xacro:front_wheel_lr>
+  <xacro:front_wheel_lr name="front_right" parent="chassis" reflect="-1" wheel_radius="${wheel_radius}" wheel_thickness="${wheel_thickness}" wheel_mass="${wheel_mass}" steer_radius="${steer_radius}" steer_thickness="${steer_thickness}" steer_mass="${steer_mass}" base_length="${base_length}" base_width="${base_width}" axle_offset="${axle_offset}" steer_height="${wheel_radius+steer_offset}"></xacro:front_wheel_lr>
+  <xacro:front_wheel_lr name="front_left" parent="chassis" reflect="1" wheel_radius="${wheel_radius}" wheel_thickness="${wheel_thickness}" wheel_mass="${wheel_mass}" steer_radius="${steer_radius}" steer_thickness="${steer_thickness}" steer_mass="${steer_mass}" base_length="${base_length}" base_width="${base_width}" axle_offset="${axle_offset}" steer_height="${wheel_radius+steer_offset}"></xacro:front_wheel_lr>
   <!-- Rear wheels -->
-  <xacro:rear_wheel_lr
-    name="rear_right"
-    parent="base"
-    wheel_radius="${wheel_radius}"
-    wheel_thickness="${wheel_thickness}"
-    wheel_mass="${wheel_mass}">
-    <origin xyz="${-base_length/2+axle_offset} ${-base_width/2-axle_offset} 0" rpy="${-90 * deg_to_rad} 0 0"/>
+  <xacro:rear_wheel_lr name="rear_right" parent="chassis" wheel_radius="${wheel_radius}" wheel_thickness="${wheel_thickness}" wheel_mass="${wheel_mass}">
+    <origin xyz="${-base_length/2+axle_offset} ${-base_width/2-axle_offset} 0" rpy="${-90 * deg_to_rad} 0 0" />
   </xacro:rear_wheel_lr>
-  <xacro:rear_wheel_lr
-    name="rear_left"
-    parent="base"
-    wheel_radius="${wheel_radius}"
-    wheel_thickness="${wheel_thickness}"
-    wheel_mass="${wheel_mass}">
-    <origin xyz="${-base_length/2+axle_offset} ${+base_width/2+axle_offset} 0" rpy="${-90 * deg_to_rad} 0 0"/>
+  <xacro:rear_wheel_lr name="rear_left" parent="chassis" wheel_radius="${wheel_radius}" wheel_thickness="${wheel_thickness}" wheel_mass="${wheel_mass}">
+    <origin xyz="${-base_length/2+axle_offset} ${+base_width/2+axle_offset} 0" rpy="${-90 * deg_to_rad} 0 0" />
   </xacro:rear_wheel_lr>
   <!-- Colour -->

File: steer_bot_description/urdf/wheel.xacro (robot description, xacro)
@@ -58,5 +58,5 @@
       <type>transmission_interface/SimpleTransmission</type>
       <actuator name="${name}_steer_joint_motor">
-        <mechanicalReduction>1</mechanicalReduction>
+        <mechanicalReduction>20</mechanicalReduction>
         <hardwareInterface>hardware_interface/PositionJointInterface</hardwareInterface>
       </actuator>
@@ -141,5 +141,5 @@
       <type>transmission_interface/SimpleTransmission</type>
       <actuator name="${name}_steer_joint_motor">
-        <mechanicalReduction>1</mechanicalReduction>
+        <mechanicalReduction>20</mechanicalReduction>
         <hardwareInterface>hardware_interface/PositionJointInterface</hardwareInterface>
       </actuator>
@@ -213,6 +213,6 @@
     </gazebo>
   </xacro:macro>
-  <!-- Bicycle model front wheel link (passive - no transmission) -->
-  <xacro:macro name="front_wheel"
+  <!-- Car steering model rear wheel links (left/right) -->
+  <xacro:macro name="rear_wheel_lr"
     params="
       name
@@ -228,5 +228,5 @@
           <cylinder radius="${wheel_radius}" length="${wheel_thickness}"/>
         </geometry>
-        <material name="yellow" />
+        <material name="red" />
       </visual>
       <collision>
@@ -247,45 +247,4 @@
       <axis xyz="0 0 1"/>
     </joint>
-    <gazebo reference="${name}_wheel_link">
-      <material>Gazebo/Yellow</material>
-    </gazebo>
-    <gazebo reference="${name}_wheel_joint">
-      <provideFeedback>true</provideFeedback>
-    </gazebo>
-  </xacro:macro>
-  <!-- Car steering model rear wheel links (left/right) -->
-  <xacro:macro name="rear_wheel_lr"
-    params="
-      name
-      parent
-      wheel_radius
-      wheel_thickness
-      wheel_mass
-      *origin">
-    <link name="${name}_wheel_link">
-      <visual>
-        <origin xyz="0 0 0" rpy="0 0 0"/>
-        <geometry>
-          <cylinder radius="${wheel_radius}" length="${wheel_thickness}"/>
-        </geometry>
-        <material name="red" />
-      </visual>
-      <collision>
-        <origin xyz="0 0 0" rpy="0 0 0"/>
-        <geometry>
-          <cylinder radius="${wheel_radius}" length="${wheel_thickness}"/>
-        </geometry>
-      </collision>
-      <xacro:solid_cylinder_inertial
-          rpy="0 0 0" xyz="0 0 0"
-          mass="${wheel_mass}"
-          radius="${wheel_radius}" length="${wheel_thickness}" />
-    </link>
-    <joint name="${name}_wheel_joint" type="continuous">
-      <parent link="${parent}_link"/>
-      <child link="${name}_wheel_link"/>
-      <xacro:insert_block name="origin"/>
-      <axis xyz="0 0 1"/>
-    </joint>
     <transmission name="${name}_wheel_joint_trans">
       <type>transmission_interface/SimpleTransmission</type>

Commit message: -remove bicycle model something broken

File: steer_bot_description/urdf/steer_bot.urdf.xacro (robot description, xacro)
@@ -16,6 +16,6 @@
 <robot name="steer_bot" xmlns:xacro="http://wiki.ros.org/xacro">
   <!-- Include xacro for inertials, materials and wheels -->
-  <xacro:include filename="$(find steer_bot_description)/urdf/wheel.xacro"/>
-  <xacro:property name="robot_namespace" value="/steer_bot"/>
+  <xacro:include filename="$(find steer_bot_description)/urdf/wheel.xacro" />
+  <xacro:property name="robot_namespace" value="/steer_bot" />
   <!-- Gazebo plugins -->
   <gazebo>
@@ -27,110 +27,66 @@
       <legacyModeNS>false</legacyModeNS>
     </plugin>
+    <plugin name="p3d_base_controller" filename="libgazebo_ros_p3d.so">
+      <alwaysOn>true</alwaysOn>
+      <updateRate>50.0</updateRate>
+      <bodyName>base_link</bodyName>
+      <topicName>odom</topicName>
+      <gaussianNoise>0.01</gaussianNoise>
+      <frameName>world</frameName>
+      <xyzOffsets>0 0 0</xyzOffsets>
+      <rpyOffsets>0 0 0</rpyOffsets>
+    </plugin>
   </gazebo>
   <!-- Math constants -->
-  <xacro:property name="deg_to_rad" value="0.01745329251994329577"/>
+  <xacro:property name="deg_to_rad" value="0.01745329251994329577" />
   <!-- Robot base dimensions -->
-  <xacro:property name="base_length" value="0.5" />
-  <xacro:property name="base_width" value="0.3" />
+  <xacro:property name="base_length" value="3.6" />
+  <xacro:property name="base_width" value="2.5" />
   <xacro:property name="base_height" value="0.1" />
-  <xacro:property name="base_mass" value="5" />
+  <xacro:property name="base_mass" value="8000" />
   <!-- Wheel link dimensions -->
-  <xacro:property name="wheel_radius" value="0.1" />
-  <xacro:property name="wheel_thickness" value="0.08" />
-  <xacro:property name="wheel_mass" value="1" />
+  <xacro:property name="wheel_radius" value="0.5" />
+  <xacro:property name="wheel_thickness" value="0.3" />
+  <xacro:property name="wheel_mass" value="100" />
   <!-- Steering link dimensions -->
-  <xacro:property name="steer_radius" value="0.05" />
-  <xacro:property name="steer_thickness" value="0.02" />
-  <xacro:property name="steer_mass" value="1" />
+  <xacro:property name="steer_radius" value="0.1" />
+  <xacro:property name="steer_thickness" value="0.5" />
+  <xacro:property name="steer_mass" value="10" />
   <!-- Axle positions -->
-  <xacro:property name="axle_offset" value="0.05" />
-  <xacro:property name="steer_offset" value="0.02" />
+  <xacro:property name="axle_offset" value="0.275" />
+  <xacro:property name="steer_offset" value="0.1" />
   <!-- Base link -->
-  <link name="base_link">
+  <link name="base_link"></link>
+  <!-- A fixed joint for to connect base and chassis links -->
+  <joint name="base_link" type="fixed">
+    <origin xyz="0 0 0" rpy="0 0 0" />
+    <parent link="base_link" />
+    <child link="chassis_link" />
+  </joint>
+  <!-- Dummy Chassis link -->
+  <link name="chassis_link">
     <visual>
-      <origin xyz="0 0 0" rpy="0 0 0"/>
+      <origin xyz="0 0 0" rpy="0 0 0" />
       <geometry>
-        <box size="${base_length} ${base_width} ${base_height}"/>
+        <box size="${base_length} ${base_width} ${base_height}" />
       </geometry>
       <material name="green" />
     </visual>
-    <collision>
-      <origin xyz="0 0 0" rpy="0 0 0"/>
-      <geometry>
-        <box size="${base_length} ${base_width} ${base_height}"/>
-      </geometry>
-    </collision>
-    <xacro:solid_cuboid_inertial
-        rpy="0 0 0" xyz="0 0 0"
-        mass="${base_mass}"
-        x="${base_length}" y="${base_width}" z="${base_height}" />
+    <xacro:solid_cuboid_inertial rpy="0 0 0" xyz="0 0 0" mass="${base_mass}" x="${base_length}" y="${base_width}" z="${base_height}" />
   </link>
   <!-- Front steer and rear wheel joints required for ackermann_steering_controller -->
-  <xacro:front_steer
-    name="front"
-    parent="base"
-    steer_radius="${steer_radius}"
-    steer_thickness="${steer_thickness}"
-    steer_mass="${steer_mass}"
-    base_length="${base_length}"
-    base_width="${base_width}"
-    axle_offset="${axle_offset}"
-    steer_height="${wheel_radius+steer_offset}">
-  </xacro:front_steer>
-  <xacro:rear_wheel
-    name="rear"
-    parent="base"
-    wheel_radius="${wheel_radius/4}"
-    wheel_thickness="${wheel_thickness/2}"
-    wheel_mass="${wheel_mass/32}">
-    <origin xyz="${-base_length/2+axle_offset} 0 0" rpy="${-90 * deg_to_rad} 0 0"/>
+  <xacro:front_steer name="front" parent="chassis" steer_radius="${steer_radius}" steer_thickness="${steer_thickness}" steer_mass="${steer_mass}" base_length="${base_length}" base_width="${base_width}" axle_offset="${axle_offset}" steer_height="${wheel_radius+steer_offset}"></xacro:front_steer>
+  <xacro:rear_wheel name="rear" parent="chassis" wheel_radius="${wheel_radius/4}" wheel_thickness="${wheel_thickness/2}" wheel_mass="${wheel_mass/32}">
+    <origin xyz="${-base_length/2+axle_offset} 0 0" rpy="${-90 * deg_to_rad} 0 0" />
   </xacro:rear_wheel>
   <!-- Steerable front wheels -->
-  <xacro:front_wheel_lr
-    name="front_right"
-    parent="base"
-    reflect="-1"
-    wheel_radius="${wheel_radius}"
-    wheel_thickness="${wheel_thickness}"
-    wheel_mass="${wheel_mass}"
-    steer_radius="${steer_radius}"
-    steer_thickness="${steer_thickness}"
-    steer_mass="${steer_mass}"
-    base_length="${base_length}"
-    base_width="${base_width}"
-    axle_offset="${axle_offset}"
-    steer_height="${wheel_radius+steer_offset}">
-  </xacro:front_wheel_lr>
-  <xacro:front_wheel_lr
-    name="front_left"
-    parent="base"
-    reflect="1"
-    wheel_radius="${wheel_radius}"
-    wheel_thickness="${wheel_thickness}"
-    wheel_mass="${wheel_mass}"
-    steer_radius="${steer_radius}"
-    steer_thickness="${steer_thickness}"
-    steer_mass="${steer_mass}"
-    base_length="${base_length}"
-    base_width="${base_width}"
-    axle_offset="${axle_offset}"
-    steer_height="${wheel_radius+steer_offset}">
-  </xacro:front_wheel_lr>
+  <xacro:front_wheel_lr name="front_right" parent="chassis" reflect="-1" wheel_radius="${wheel_radius}" wheel_thickness="${wheel_thickness}" wheel_mass="${wheel_mass}" steer_radius="${steer_radius}" steer_thickness="${steer_thickness}" steer_mass="${steer_mass}" base_length="${base_length}" base_width="${base_width}" axle_offset="${axle_offset}" steer_height="${wheel_radius+steer_offset}"></xacro:front_wheel_lr>
+  <xacro:front_wheel_lr name="front_left" parent="chassis" reflect="1" wheel_radius="${wheel_radius}" wheel_thickness="${wheel_thickness}" wheel_mass="${wheel_mass}" steer_radius="${steer_radius}" steer_thickness="${steer_thickness}" steer_mass="${steer_mass}" base_length="${base_length}" base_width="${base_width}" axle_offset="${axle_offset}" steer_height="${wheel_radius+steer_offset}"></xacro:front_wheel_lr>
   <!-- Rear wheels -->
-  <xacro:rear_wheel_lr
-    name="rear_right"
-    parent="base"
-    wheel_radius="${wheel_radius}"
-    wheel_thickness="${wheel_thickness}"
-    wheel_mass="${wheel_mass}">
-    <origin xyz="${-base_length/2+axle_offset} ${-base_width/2-axle_offset} 0" rpy="${-90 * deg_to_rad} 0 0"/>
+  <xacro:rear_wheel_lr name="rear_right" parent="chassis" wheel_radius="${wheel_radius}" wheel_thickness="${wheel_thickness}" wheel_mass="${wheel_mass}">
+    <origin xyz="${-base_length/2+axle_offset} ${-base_width/2-axle_offset} 0" rpy="${-90 * deg_to_rad} 0 0" />
   </xacro:rear_wheel_lr>
-  <xacro:rear_wheel_lr
-    name="rear_left"
-    parent="base"
-    wheel_radius="${wheel_radius}"
-    wheel_thickness="${wheel_thickness}"
-    wheel_mass="${wheel_mass}">
-    <origin xyz="${-base_length/2+axle_offset} ${+base_width/2+axle_offset} 0" rpy="${-90 * deg_to_rad} 0 0"/>
+  <xacro:rear_wheel_lr name="rear_left" parent="chassis" wheel_radius="${wheel_radius}" wheel_thickness="${wheel_thickness}" wheel_mass="${wheel_mass}">
+    <origin xyz="${-base_length/2+axle_offset} ${+base_width/2+axle_offset} 0" rpy="${-90 * deg_to_rad} 0 0" />
   </xacro:rear_wheel_lr>
   <!-- Colour -->

File: steer_bot_description/urdf/wheel.xacro (robot description, xacro)
@@ -12,5 +12,5 @@
   <xacro:include filename="$(find steer_bot_description)/urdf/inertials.xacro"/>
   <!-- Properties -->
-  <xacro:property name="steer_effort" value="10.0"/>
+  <xacro:property name="steer_effort" value="100.0"/>
   <xacro:property name="steer_velocity" value="5.0"/>
   <xacro:property name="steer_limit_deg" value="45.0"/>
@@ -58,5 +58,5 @@
       <type>transmission_interface/SimpleTransmission</type>
       <actuator name="${name}_steer_joint_motor">
-        <mechanicalReduction>1</mechanicalReduction>
+        <mechanicalReduction>20</mechanicalReduction>
         <hardwareInterface>hardware_interface/PositionJointInterface</hardwareInterface>
       </actuator>
@@ -141,5 +141,5 @@
       <type>transmission_interface/SimpleTransmission</type>
       <actuator name="${name}_steer_joint_motor">
-        <mechanicalReduction>1</mechanicalReduction>
+        <mechanicalReduction>20</mechanicalReduction>
         <hardwareInterface>hardware_interface/PositionJointInterface</hardwareInterface>
       </actuator>
@@ -213,45 +213,45 @@
     </gazebo>
   </xacro:macro>
-  <!-- Bicycle model front wheel link (passive - no transmission) -->
-  <xacro:macro name="front_wheel"
-    params="
-      name
-      parent
-      wheel_radius
-      wheel_thickness
-      wheel_mass
-      *origin">
-    <link name="${name}_wheel_link">
-      <visual>
-        <origin xyz="0 0 0" rpy="0 0 0"/>
-        <geometry>
-          <cylinder radius="${wheel_radius}" length="${wheel_thickness}"/>
-        </geometry>
-        <material name="yellow" />
-      </visual>
-      <collision>
-        <origin xyz="0 0 0" rpy="0 0 0"/>
-        <geometry>
-          <cylinder radius="${wheel_radius}" length="${wheel_thickness}"/>
-        </geometry>
-      </collision>
-      <xacro:solid_cylinder_inertial
-          rpy="0 0 0" xyz="0 0 0"
-          mass="${wheel_mass}"
-          radius="${wheel_radius}" length="${wheel_thickness}" />
-    </link>
-    <joint name="${name}_wheel_joint" type="continuous">
-      <parent link="${parent}_link"/>
-      <child link="${name}_wheel_link"/>
-      <xacro:insert_block name="origin"/>
-      <axis xyz="0 0 1"/>
-    </joint>
-    <gazebo reference="${name}_wheel_link">
-      <material>Gazebo/Yellow</material>
-    </gazebo>
-    <gazebo reference="${name}_wheel_joint">
-      <provideFeedback>true</provideFeedback>
-    </gazebo>
-  </xacro:macro>
+   <!-- Bicycle model front wheel link (passive - no transmission) -->
+   <xacro:macro name="front_wheel"
+   params="
+     name
+     parent
+     wheel_radius
+     wheel_thickness
+     wheel_mass
+     *origin">
+   <link name="${name}_wheel_link">
+     <visual>
+       <origin xyz="0 0 0" rpy="0 0 0"/>
+       <geometry>
+         <cylinder radius="${wheel_radius}" length="${wheel_thickness}"/>
+       </geometry>
+       <material name="yellow" />
+     </visual>
+     <collision>
+       <origin xyz="0 0 0" rpy="0 0 0"/>
+       <geometry>
+         <cylinder radius="${wheel_radius}" length="${wheel_thickness}"/>
+       </geometry>
+     </collision>
+     <xacro:solid_cylinder_inertial
+         rpy="0 0 0" xyz="0 0 0"
+         mass="${wheel_mass}"
+         radius="${wheel_radius}" length="${wheel_thickness}" />
+   </link>
+   <joint name="${name}_wheel_joint" type="continuous">
+     <parent link="${parent}_link"/>
+     <child link="${name}_wheel_link"/>
+     <xacro:insert_block name="origin"/>
+     <axis xyz="0 0 1"/>
+   </joint>
+   <gazebo reference="${name}_wheel_link">
+     <material>Gazebo/Yellow</material>
+   </gazebo>
+   <gazebo reference="${name}_wheel_joint">
+     <provideFeedback>true</provideFeedback>
+   </gazebo>
+ </xacro:macro>
   <!-- Car steering model rear wheel links (left/right) -->
   <xacro:macro name="rear_wheel_lr"
