Commit message: simulation changes

File: steer_bot_description/urdf/steer_bot.urdf.xacro (robot description, xacro)
@@ -27,4 +27,5 @@
       <legacyModeNS>false</legacyModeNS>
     </plugin>
+    <!-- <plugin name="disable_physics" filename="libdisable_plugin.so" /> -->
     <plugin name="p3d_base_controller" filename="libgazebo_ros_p3d.so">
       <alwaysOn>true</alwaysOn>
@@ -33,5 +34,5 @@
       <topicName>odom</topicName>
       <gaussianNoise>0.01</gaussianNoise>
-      <frameName>world</frameName>
+      <frameName>map</frameName>
       <xyzOffsets>0 0 0</xyzOffsets>
       <rpyOffsets>0 0 0</rpyOffsets>
@@ -44,18 +45,20 @@
   <xacro:property name="base_width" value="2.5" />
   <xacro:property name="base_height" value="0.1" />
-  <xacro:property name="base_mass" value="8000" />
+  <xacro:property name="base_mass" value="0.0001" />
   <!-- Wheel link dimensions -->
   <xacro:property name="wheel_radius" value="0.5" />
   <xacro:property name="wheel_thickness" value="0.3" />
-  <xacro:property name="wheel_mass" value="100" />
+  <xacro:property name="wheel_mass" value="0.0001" />
   <!-- Steering link dimensions -->
   <xacro:property name="steer_radius" value="0.1" />
   <xacro:property name="steer_thickness" value="0.5" />
-  <xacro:property name="steer_mass" value="10" />
+  <xacro:property name="steer_mass" value="0.0001" />
   <!-- Axle positions -->
   <xacro:property name="axle_offset" value="0.275" />
   <xacro:property name="steer_offset" value="0.1" />
   <!-- Base link -->
-  <link name="base_link"></link>
+  <link name="base_link">
+    <kinematic>true</kinematic>
+  </link>
   <!-- A fixed joint for to connect base and chassis links -->
   <joint name="base_link" type="fixed">
@@ -97,6 +100,16 @@
   </xacro:rear_wheel_lr>
   <!-- Colour -->
+  <gazebo reference="chassis_link">
+    <material>Gazebo/Green</material>
+    <velocity_decay>
+      <linear>0.5</linear>
+      <angular>0.5</angular>
+    </velocity_decay>
+  </gazebo>
   <gazebo reference="base_link">
-    <material>Gazebo/Green</material>
+    <velocity_decay>
+      <linear>0.5</linear>
+      <angular>0.5</angular>
+    </velocity_decay>
   </gazebo>
 </robot>

File: steer_bot_description/urdf/wheel.xacro (robot description, xacro)
@@ -9,13 +9,12 @@
 <robot name="wheel" xmlns:xacro="http://wiki.ros.org/xacro">
   <!-- Include xacro for materials and inertials -->
-  <xacro:include filename="$(find steer_bot_description)/urdf/materials.xacro"/>
-  <xacro:include filename="$(find steer_bot_description)/urdf/inertials.xacro"/>
+  <xacro:include filename="$(find steer_bot_description)/urdf/materials.xacro" />
+  <xacro:include filename="$(find steer_bot_description)/urdf/inertials.xacro" />
   <!-- Properties -->
-  <xacro:property name="steer_effort" value="100.0"/>
-  <xacro:property name="steer_velocity" value="5.0"/>
-  <xacro:property name="steer_limit_deg" value="45.0"/>
+  <xacro:property name="steer_effort" value="100.0" />
+  <xacro:property name="steer_velocity" value="5.0" />
+  <xacro:property name="steer_limit_deg" value="45.0" />
   <!-- Bicycle model front steering link (required for steer_drive_controller) -->
-  <xacro:macro name="front_steer"
-    params="
+  <xacro:macro name="front_steer" params="
       name
       parent
@@ -28,35 +27,41 @@
       steer_height">
     <link name="${name}_steer_link">
-      <visual>
-        <origin xyz="0 0 0" rpy="0 0 0"/>
-        <geometry>
-          <cylinder radius="${steer_radius}" length="${steer_thickness}"/>
+      <kinematic>true</kinematic>
+      <visual>
+        <origin xyz="0 0 0" rpy="0 0 0" />
+        <geometry>
+          <cylinder radius="${steer_radius}" length="${steer_thickness}" />
         </geometry>
         <material name="yellow" />
       </visual>
       <collision>
-        <origin xyz="0 0 0" rpy="0 0 0"/>
-        <geometry>
-          <cylinder radius="${steer_radius}" length="${steer_thickness}"/>
-        </geometry>
-      </collision>
-      <xacro:solid_cylinder_inertial
-          rpy="0 0 0" xyz="0 0 0"
-          mass="${steer_mass}"
-          radius="${steer_radius}" length="${steer_thickness}" />
+        <origin xyz="0 0 0" rpy="0 0 0" />
+        <geometry>
+          <cylinder radius="${steer_radius}" length="${steer_thickness}" />
+        </geometry>
+        <surface>
+          <friction>
+            <ode>
+              <mu>10000000.0</mu>
+              <mu2>10000000.0</mu2>
+              <slip1>0.0</slip1>
+              <slip2>0.0</slip2>
+            </ode>
+          </friction>
+        </surface>
+      </collision>
+      <xacro:solid_cylinder_inertial rpy="0 0 0" xyz="0 0 0" mass="${steer_mass}" radius="${steer_radius}" length="${steer_thickness}" />
     </link>
     <joint name="${name}_steer_joint" type="revolute">
-      <parent link="${parent}_link"/>
-      <child link="${name}_steer_link"/>
-      <origin xyz="${base_length/2-axle_offset} 0 ${steer_height}" rpy="0 0 0"/>
-      <axis xyz="0 0 1"/>
-      <limit effort="${steer_effort}"
-             lower="${-180.0 * deg_to_rad}" upper="${180.0 * deg_to_rad}"
-             velocity="${steer_velocity}"/>
+      <parent link="${parent}_link" />
+      <child link="${name}_steer_link" />
+      <origin xyz="${base_length/2-axle_offset} 0 ${steer_height}" rpy="0 0 0" />
+      <axis xyz="0 0 1" />
+      <limit effort="${steer_effort}" lower="${-180.0 * deg_to_rad}" upper="${180.0 * deg_to_rad}" velocity="${steer_velocity}" />
     </joint>
     <transmission name="${name}_steer_joint_trans">
       <type>transmission_interface/SimpleTransmission</type>
       <actuator name="${name}_steer_joint_motor">
-        <mechanicalReduction>20</mechanicalReduction>
+        <mechanicalReduction>1</mechanicalReduction>
         <hardwareInterface>hardware_interface/PositionJointInterface</hardwareInterface>
       </actuator>
@@ -70,6 +75,5 @@
   </xacro:macro>
   <!-- Car steering model front (steerable) wheel links (left/right) -->
-  <xacro:macro name="front_wheel_lr"
-    params="
+  <xacro:macro name="front_wheel_lr" params="
       name
       parent
@@ -86,60 +90,75 @@
       steer_height">
     <link name="${name}_steer_link">
-      <visual>
-        <origin xyz="0 0 0" rpy="0 0 0"/>
-        <geometry>
-          <cylinder radius="${steer_radius}" length="${steer_thickness}"/>
+      <kinematic>true</kinematic>
+      <visual>
+        <origin xyz="0 0 0" rpy="0 0 0" />
+        <geometry>
+          <cylinder radius="${steer_radius}" length="${steer_thickness}" />
         </geometry>
         <material name="blue" />
       </visual>
       <collision>
-        <origin xyz="0 0 0" rpy="0 0 0"/>
-        <geometry>
-          <cylinder radius="${steer_radius}" length="${steer_thickness}"/>
-        </geometry>
-      </collision>
-      <xacro:solid_cylinder_inertial
-          rpy="0 0 0" xyz="0 0 0"
-          mass="${steer_mass}"
-          radius="${steer_radius}" length="${steer_thickness}" />
+        <origin xyz="0 0 0" rpy="0 0 0" />
+        <geometry>
+          <cylinder radius="${steer_radius}" length="${steer_thickness}" />
+        </geometry>
+        <surface>
+          <friction>
+            <ode>
+              <mu>10000000.0</mu>
+              <mu2>10000000.0</mu2>
+              <slip1>0.0</slip1>
+              <slip2>0.0</slip2>
+            </ode>
+          </friction>
+        </surface>
+      </collision>
+      <xacro:solid_cylinder_inertial rpy="0 0 0" xyz="0 0 0" mass="${steer_mass}" radius="${steer_radius}" length="${steer_thickness}" />
     </link>
     <joint name="${name}_steer_joint" type="revolute">
-      <parent link="${parent}_link"/>
-      <child link="${name}_steer_link"/>
-      <origin xyz="${base_length/2-axle_offset} ${reflect*(base_width/2+axle_offset)} ${steer_height}" rpy="0 0 0"/>
-      <axis xyz="0 0 1"/>
-      <limit effort="${steer_effort}"
-             lower="${steer_limit_deg * deg_to_rad * -1.0}" upper="${steer_limit_deg * deg_to_rad}"
-             velocity="${steer_velocity}"/>
+      <parent link="${parent}_link" />
+      <child link="${name}_steer_link" />
+      <origin xyz="${base_length/2-axle_offset} ${reflect*(base_width/2+axle_offset)} ${steer_height}" rpy="0 0 0" />
+      <axis xyz="0 0 1" />
+      <limit effort="${steer_effort}" lower="${steer_limit_deg * deg_to_rad * -1.0}" upper="${steer_limit_deg * deg_to_rad}" velocity="${steer_velocity}" />
     </joint>
     <link name="${name}_wheel_link">
-      <visual>
-        <origin xyz="0 0 0" rpy="0 0 0"/>
-        <geometry>
-          <cylinder radius="${wheel_radius}" length="${wheel_thickness}"/>
+      <kinematic>true</kinematic>
+      <visual>
+        <origin xyz="0 0 0" rpy="0 0 0" />
+        <geometry>
+          <cylinder radius="${wheel_radius}" length="${wheel_thickness}" />
         </geometry>
         <material name="red" />
       </visual>
       <collision>
-        <origin xyz="0 0 0" rpy="0 0 0"/>
-        <geometry>
-          <cylinder radius="${wheel_radius}" length="${wheel_thickness}"/>
-        </geometry>
-      </collision>
-      <xacro:solid_cylinder_inertial
-          rpy="0 0 0" xyz="0 0 0"
-          mass="${wheel_mass}"
-          radius="${wheel_radius}" length="${wheel_thickness}" />
+        <origin xyz="0 0 0" rpy="0 0 0" />
+        <geometry>
+          <cylinder radius="${wheel_radius}" length="${wheel_thickness}" />
+        </geometry>
+        <surface>
+          <friction>
+            <ode>
+              <mu>10000000.0</mu>
+              <mu2>10000000.0</mu2>
+              <slip1>0.0</slip1>
+              <slip2>0.0</slip2>
+            </ode>
+          </friction>
+        </surface>
+      </collision>
+      <xacro:solid_cylinder_inertial rpy="0 0 0" xyz="0 0 0" mass="${wheel_mass}" radius="${wheel_radius}" length="${wheel_thickness}" />
     </link>
     <joint name="${name}_wheel_joint" type="continuous">
-      <parent link="${name}_steer_link"/>
-      <child link="${name}_wheel_link"/>
-      <origin xyz="0 0 ${-steer_height}" rpy="${-90 * deg_to_rad} 0 0"/>
-      <axis xyz="0 0 1"/>
+      <parent link="${name}_steer_link" />
+      <child link="${name}_wheel_link" />
+      <origin xyz="0 0 ${-steer_height}" rpy="${-90 * deg_to_rad} 0 0" />
+      <axis xyz="0 0 1" />
+      <joint_properties damping="1000.0" friction="1000.0" />
     </joint>
     <transmission name="${name}_steer_joint_trans">
       <type>transmission_interface/SimpleTransmission</type>
       <actuator name="${name}_steer_joint_motor">
-        <mechanicalReduction>20</mechanicalReduction>
+        <mechanicalReduction>1</mechanicalReduction>
         <hardwareInterface>hardware_interface/PositionJointInterface</hardwareInterface>
       </actuator>
@@ -163,9 +182,14 @@
     <gazebo reference="${name}_wheel_link">
       <material>Gazebo/Red</material>
+      <minDepth>0.005</minDepth>
+			<mu value="10000000.0"/>
+			<mu2 value="1.0"/>
+			<kp value="10000000.0" />
+			<kd value="1.0" />
+			<fdir1 value="1 0 0"/>
     </gazebo>
   </xacro:macro>
   <!-- Bicycle model rear wheel link (required for steer_drive_controller) -->
-  <xacro:macro name="rear_wheel"
-    params="
+  <xacro:macro name="rear_wheel" params="
       name
       parent
@@ -175,27 +199,40 @@
       *origin">
     <link name="${name}_wheel_link">
-      <visual>
-        <origin xyz="0 0 0" rpy="0 0 0"/>
-        <geometry>
-          <cylinder radius="${wheel_radius}" length="${wheel_thickness}"/>
+      <kinematic>true</kinematic>
+      <velocity_decay>
+        <linear>100</linear>
+        <angular>100</angular>
+      </velocity_decay>
+      <visual>
+        <origin xyz="0 0 0" rpy="0 0 0" />
+        <geometry>
+          <cylinder radius="${wheel_radius}" length="${wheel_thickness}" />
         </geometry>
         <material name="yellow" />
       </visual>
       <collision>
-        <origin xyz="0 0 0" rpy="0 0 0"/>
-        <geometry>
-          <cylinder radius="${wheel_radius}" length="${wheel_thickness}"/>
-        </geometry>
-      </collision>
-      <xacro:solid_cylinder_inertial
-          rpy="0 0 0" xyz="0 0 0"
-          mass="${wheel_mass}"
-          radius="${wheel_radius}" length="${wheel_thickness}" />
+        <origin xyz="0 0 0" rpy="0 0 0" />
+        <geometry>
+          <cylinder radius="${wheel_radius}" length="${wheel_thickness}" />
+        </geometry>
+        <surface>
+          <friction>
+            <ode>
+              <mu>10000000.0</mu>
+              <mu2>10000000.0</mu2>
+              <slip1>0.0</slip1>
+              <slip2>0.0</slip2>
+            </ode>
+          </friction>
+        </surface>
+      </collision>
+      <xacro:solid_cylinder_inertial rpy="0 0 0" xyz="0 0 0" mass="${wheel_mass}" radius="${wheel_radius}" length="${wheel_thickness}" />
     </link>
     <joint name="${name}_wheel_joint" type="continuous">
-      <parent link="${parent}_link"/>
-      <child link="${name}_wheel_link"/>
-      <xacro:insert_block name="origin"/>
-      <axis xyz="0 0 1"/>
+      <parent link="${parent}_link" />
+      <child link="${name}_wheel_link" />
+      <xacro:insert_block name="origin" />
+      <axis xyz="0 0 1" />
+      <joint_properties damping="1000.0" friction="1000.0" />
     </joint>
     <transmission name="${name}_wheel_joint_trans">
@@ -211,9 +248,14 @@
     <gazebo reference="${name}_wheel_link">
       <material>Gazebo/Yellow</material>
-    </gazebo>
-  </xacro:macro>
-   <!-- Bicycle model front wheel link (passive - no transmission) -->
-   <xacro:macro name="front_wheel"
-   params="
+      <minDepth>0.005</minDepth>
+			<mu value="10000000.0"/>
+			<mu2 value="1.0"/>
+			<kp value="10000000.0" />
+			<kd value="1.0" />
+			<fdir1 value="1 0 0"/>
+    </gazebo>
+  </xacro:macro>
+  <!-- Bicycle model front wheel link (passive - no transmission) -->
+  <xacro:macro name="front_wheel" params="
      name
      parent
@@ -222,39 +264,52 @@
      wheel_mass
      *origin">
-   <link name="${name}_wheel_link">
-     <visual>
-       <origin xyz="0 0 0" rpy="0 0 0"/>
-       <geometry>
-         <cylinder radius="${wheel_radius}" length="${wheel_thickness}"/>
-       </geometry>
-       <material name="yellow" />
-     </visual>
-     <collision>
-       <origin xyz="0 0 0" rpy="0 0 0"/>
-       <geometry>
-         <cylinder radius="${wheel_radius}" length="${wheel_thickness}"/>
-       </geometry>
-     </collision>
-     <xacro:solid_cylinder_inertial
-         rpy="0 0 0" xyz="0 0 0"
-         mass="${wheel_mass}"
-         radius="${wheel_radius}" length="${wheel_thickness}" />
-   </link>
-   <joint name="${name}_wheel_joint" type="continuous">
-     <parent link="${parent}_link"/>
-     <child link="${name}_wheel_link"/>
-     <xacro:insert_block name="origin"/>
-     <axis xyz="0 0 1"/>
-   </joint>
-   <gazebo reference="${name}_wheel_link">
-     <material>Gazebo/Yellow</material>
-   </gazebo>
-   <gazebo reference="${name}_wheel_joint">
-     <provideFeedback>true</provideFeedback>
-   </gazebo>
- </xacro:macro>
+    <link name="${name}_wheel_link">
+      <kinematic>true</kinematic>
+      <visual>
+        <origin xyz="0 0 0" rpy="0 0 0" />
+        <geometry>
+          <cylinder radius="${wheel_radius}" length="${wheel_thickness}" />
+        </geometry>
+        <material name="yellow" />
+      </visual>
+      <collision>
+        <origin xyz="0 0 0" rpy="0 0 0" />
+        <geometry>
+          <cylinder radius="${wheel_radius}" length="${wheel_thickness}" />
+        </geometry>
+        <surface>
+          <friction>
+            <ode>
+              <mu>10000000.0</mu>
+              <mu2>10000000.0</mu2>
+              <slip1>0.0</slip1>
+              <slip2>0.0</slip2>
+            </ode>
+          </friction>
+        </surface>
+      </collision>
+      <xacro:solid_cylinder_inertial rpy="0 0 0" xyz="0 0 0" mass="${wheel_mass}" radius="${wheel_radius}" length="${wheel_thickness}" />
+    </link>
+    <joint name="${name}_wheel_joint" type="continuous">
+      <parent link="${parent}_link" />
+      <child link="${name}_wheel_link" />
+      <xacro:insert_block name="origin" />
+      <axis xyz="0 0 1" />
+    </joint>
+    <gazebo reference="${name}_wheel_link">
+      <material>Gazebo/Yellow</material>
+      <minDepth>0.005</minDepth>
+      <mu value="10000000.0" />
+      <mu2 value="10000000.0" />
+      <kp value="10000000.0" />
+      <kd value="1.0" />
+      <fdir1 value="1 0 0" />
+    </gazebo>
+    <gazebo reference="${name}_wheel_joint">
+      <provideFeedback>true</provideFeedback>
+    </gazebo>
+  </xacro:macro>
   <!-- Car steering model rear wheel links (left/right) -->
-  <xacro:macro name="rear_wheel_lr"
-    params="
+  <xacro:macro name="rear_wheel_lr" params="
       name
       parent
@@ -264,27 +319,35 @@
       *origin">
     <link name="${name}_wheel_link">
-      <visual>
-        <origin xyz="0 0 0" rpy="0 0 0"/>
-        <geometry>
-          <cylinder radius="${wheel_radius}" length="${wheel_thickness}"/>
+      <kinematic>true</kinematic>
+      <visual>
+        <origin xyz="0 0 0" rpy="0 0 0" />
+        <geometry>
+          <cylinder radius="${wheel_radius}" length="${wheel_thickness}" />
         </geometry>
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